File: Dust-Collector-Reciever.kicad_sch (KiCad schematic)
At the start: 3 parts

Commit message: WIP - around 70% done on schematic
Parts:
- added C1, C3, C5, C6: 10u, symbol Device:C
- added C2: 1u, symbol Device:C
- added C4: 0.1uf, symbol Device:C
- added H1, H2, H3, H4: MountingHole, MountingHole:MountingHole_3.2mm_M3_ISO7380_Pad, symbol Mechanical:MountingHole
- added J1, J2: Screw_Terminal_01x04, TerminalBlock_Phoenix:TerminalBlock_Phoenix_MKDS-1,5-4-5.08_1x04_P5.08mm_Horizontal, symbol Connector:Screw_Terminal_01x04
- added J3: ANT_OUT, symbol Connector:Conn_01x01_Socket
- added J4: Conn_ARM_JTAG_SWD_10, Connector_PinHeader_1.27mm:PinHeader_2x05_P1.27mm_Vertical, symbol Connector:Conn_ARM_JTAG_SWD_10
- added L1, L2: 6.8uH, symbol Device:L
- added R1: 100k, symbol Device:R
- added R2: 100, symbol Device:R
- added R3: 10k, symbol Device:R
- added SW1: SW_Push, symbol Switch:SW_Push
- added U4: CPC1006N NO, Package_SO:SO-4_4.4x4.3mm_P2.54mm, symbol Relay_SolidState:ASSR-1218
- added U5: CPC1106N NC, Package_SO:SO-4_4.4x4.3mm_P2.54mm, symbol Relay_SolidState:ASSR-1218
- added U6: AP2112K-3.3, Package_TO_SOT_SMD:SOT-23-5, symbol Regulator_Linear:AP2112K-3.3
- U1: renamed from U?; value STM32L011K3Tx -> STM32L010K4T6-ND; DigiKey (none) -> 497-STM32L010K4T6-ND
- U2: renamed from U?; now not fitted; now left out of the parts list
- gave numbers to parts that had none: 1
Connections:
- net GND: now reaches U3.1 (GND)
- net GND: now also U1.16 (VSS), U1.32 (VSS), U3.10 (GND), U3.8 (GND), C1.2, C2.2, C3.2, C4.1, C5.2, C6.2, J2.2 (Pin_2), J4.3 (GND), J4.5 (GND), J4.9 (GNDDetect), R3.2, SW1.1, U4.2, U5.2, U6.2 (GND)
- net +3V3: now reaches U3.13 (3.3V)
- net +3V3: now also U1.1 (VDD), U1.17 (VDD), U1.5 (VDDA), C2.1, C3.1, J4.1 (VTref), U6.5 (VOUT)
- net at U3.2 (MISO): now also U1.12 (PA6)
- net at U3.3 (MOSI): now also U1.13 (PA7)
- net at U3.4 (SCK): now also U1.11 (PA5)
- net at U3.5 (NSS): now also U1.25 (PA15)
- net RESET: now reaches U3.6 (RESET)
- net RESET: now also U1.4 (NRST), C4.2, J4.10 (~{RESET}), SW1.2
- net at U3.9 (ANT): now also J3.1 (Pin_1)
- net at U1.14 (PB0): now also U5.1
- net SWDIO: now reaches U1.23 (PA13)
- net SWDIO: now also J4.2 (SWDIO/TMS)
- net SWDCLK: now reaches U1.24 (PA14)
- net SWDCLK: now also J4.4 (SWDCLK/TCK)
- net at U1.26 (PB3): now also U4.1
- net LOW PASS DUSTBIN SIGNAL: now reaches U1.7 (PA1)
- net LOW PASS DUSTBIN SIGNAL: now also C6.1, L2.1
- new net: L1.2, R2.2, R3.1
- new net: C5.1, L1.1, L2.2
- new net: R1.2, U6.3 (EN)
- new net 5V0_{IN}: C1.1, J2.1 (Pin_1), R1.1, U6.1 (VIN)
- new net Common24vIN: J1.1 (Pin_1), U4.3
- new net DustBin Signal: J1.4 (Pin_4), R2.1
- new net NC/OFF Switch IN (from controller): J1.3 (Pin_3), U5.4
- new net NC/OFF Switch OUT (to switch): J1.2 (Pin_2), U5.3
- new net NO/ON Switch IN/OUT: J2.3 (Pin_3), J2.4 (Pin_4), U4.4
- new net SWO: J4.6 (SWO/TDO)
- no-connect marks 0 -> 25
Other:
- note added: "Bridges accross (parallel to) the Normally Open switch."
- note added: "Inline (series) to the Normally Closed switch."
- note added: "Power Regulation"
- note added: "Two positions provided on NO to make it easier to add the connection parallel without adding two wires to one screw terminal position. Add a jumper from one position to the switch and the other position takes the stock wire"
- moved on the sheet: U1, U3
